File: Breadboard_Power_Supply/Breadboard_Power_Supply.kicad_pcb (KiCad board)
At the start: 2 copper layers, 24.4 x 52.1 mm, 17 parts, among them J1 Barrel_Jack_Switch, J2 Conn_01x03_Pin, J3 Conn_01x02_Pin, J4 Screw_Terminal_01x02, J5 Screw_Terminal_01x02, J6 Conn_01x03_Pin, J7 Conn_01x02_Pin, SW1 SW_SPDT, U1 LM7805_TO220, U2 LM317_TO-220

Commit message: Project Completed Rev 1.0
Parts:
- added REF**: KiCad-Logo_8mm_SilkScreen, Symbol:KiCad-Logo_8mm_SilkScreen, B.Cu at (155.2, 54.8)
